Commit message: tests now compile, but they fail for some reason, and are not complete
also I updated the textures of the robot description

File: robotiq_3f_description/urdf/robotiq_3f_gripper.xacro (robot description, xacro)
@@ -1,73 +1,5 @@
 <?xml version="1.0"?>
-<robot xmlns:xacro="http://www.ros.org/wiki/xacro">
-    <xacro:include filename="$(find robotiq_3f_description)/urdf/robotiq_3f_gripper_finger_macro.xacro"/>
-    <xacro:include filename="$(find robotiq_3f_description)/urdf/robotiq_3f_driver_ros2_control.xacro"/>
-    <xacro:macro name="robotiq_3f_gripper"
-                 params="parent
-                       origin_xyz:='0 0 0'
-                       origin_rpy:='0 0 0'
-                       prefix:=''
-                       use_fake_hardware:=true
-                       usb_port:=/dev/ttyUSB0">
-        <xacro:robotiq_3f_driver_ros2_control
-                name="robotiq_3f_driver_ros2_control"
-                use_fake_hardware="${use_fake_hardware}"
-                usb_port="${usb_port}"/>
-        <xacro:robotiq_3f_gripper_finger_articulated prefix="${prefix}finger_1_"/>
-        <xacro:robotiq_3f_gripper_finger_articulated prefix="${prefix}finger_2_"/>
-        <xacro:robotiq_3f_gripper_finger_articulated prefix="${prefix}finger_middle_"/>
-        <!-- link list -->
-        <link name="${prefix}palm">
-            <visual>
-                <geometry>
-                    <mesh filename="package://robotiq_3f_description/meshes/visual/palm.dae"/>
-                </geometry>
-                <material name="gray">
-                    <color rgba="0.2 0.2 0.2 1"/>
-                </material>
-            </visual>
-            <collision>
-                <geometry>
-                    <mesh filename="package://robotiq_3f_description/meshes/collision/palm.STL"/>
-                </geometry>
-                <material name="yellow">
-                    <color rgba="0 1 1 1"/>
-                </material>
-            </collision>
-        </link>
-        <link name="${prefix}tool0"/>
-        <inertial>
-            <origin xyz="0 0 0" rpy="0 0 0"/>
-            <mass value="1.3"/>
-            <inertia ixx="0.006012" ixy="0.000079" ixz="-0.00024" iyy="0.012892" iyz="0" izz="0.002435"/>
-        </inertial>
-        <!-- end of link list -->
-        <!-- joint list -->
-        <joint name="${prefix}palm_finger_1_joint" type="revolute">
-            <parent link="${prefix}palm"/>
-            <child link="${prefix}finger_1_link_0"/>
-            <axis xyz="0 1 0"/>
-            <origin xyz="-0.0455 0.0214 0.036" rpy="0 3.1416 -1.57"/>
-            <limit lower="-0.1784" upper="0.192" effort="100" velocity="100"/>
-        </joint>
-        <joint name="${prefix}palm_finger_2_joint" type="revolute">
-            <parent link="${prefix}palm"/>
-            <child link="${prefix}finger_2_link_0"/>
-            <axis xyz="0 1 0"/>
-            <origin xyz="-0.0455 0.0214 -0.036" rpy="0 3.1416 -1.57"/>
-            <limit lower="-0.192" upper="0.1784" effort="100" velocity="100"/>
-        </joint>
-        <joint name="${prefix}palm_finger_middle_joint" type="fixed">
-            <parent link="${prefix}palm"/>
-            <child link="${prefix}finger_middle_link_0"/>
-            <axis xyz="0 0 1"/>
-            <origin xyz="0.0455 0.0214 0" rpy="0 0 1.57"/>
-        </joint>
-        <joint name="${prefix}palm_tool0" type="fixed">
-            <parent link="${prefix}palm"/>
-            <child link="${prefix}tool0"/>
-            <origin xyz="0.0 0.0875 0.0" rpy="0 0 1.5707"/>
-        </joint>
-        <!-- end of joint list -->
-    </xacro:macro>
+<robot name="example_robot" xmlns:xacro="http://www.ros.org/wiki/xacro">
+  <xacro:include filename="$(find robotiq_3f_description)/urdf/robotiq_3f_gripper_macro.xacro"/>
+  <xacro:robotiq_3f_gripper use_fake_hardware="false"/>
 </robot>

File: robotiq_3f_description/urdf/robotiq_3f_gripper_finger_macro.xacro (robot description, xacro)
@@ -14,7 +14,4 @@
                     <mesh filename="package://robotiq_3f_description/meshes/visual/link_0.dae"/>
                 </geometry>
-                <material name="gray">
-                    <color rgba="0.2 0.2 0.2 1"/>
-                </material>
             </visual>
             <collision>
@@ -39,5 +36,4 @@
                     <mesh filename="package://robotiq_3f_description/meshes/visual/link_1.dae"/>
                 </geometry>
-                <material name="gray"/>
             </visual>
             <collision>
@@ -56,5 +52,5 @@
         <link name="${prefix}link_2">
             <!--
-            NOTE: This link has an offset in the z-direction based on the models that were
+            NOTE This link has an offset in the z-direction based on the models that were
             used to generate grap-it poses.  With the offset below the model appears visually
             correct, but it is suspect.
@@ -65,5 +61,4 @@
                     <mesh filename="package://robotiq_3f_description/meshes/visual/link_2.dae"/>
                 </geometry>
-                <material name="gray"/>
             </visual>
             <collision>
@@ -86,5 +81,4 @@
                     <mesh filename="package://robotiq_3f_description/meshes/visual/link_3.dae"/>
                 </geometry>
-                <material name="gray"/>
             </visual>
             <collision>
