Commit message: working ros2 control activate and clean shutdown on CTRL+C

File: robotiq_3f_description/urdf/robotiq_3f_driver_ros2_control.xacro (robot description, xacro)
@@ -20,22 +20,60 @@
                 <param name="slave_address">${slave_address}</param>
             </hardware>
-            <joint name="finger_a">
-                <command_interface name="position"/>
+            <joint name="finger_1_joint_1">
                 <state_interface name="position"/>
-                <state_interface name="velocity"/>
-                <state_interface name="effort"/> <!-- current -->
+                <!-- NOTE should we also have position and velocity interfaces? -->
             </joint>
-            <joint name="finger_b">
-                <command_interface name="position"/>
+            <joint name="finger_1_joint_2">
                 <state_interface name="position"/>
-                <state_interface name="velocity"/>
-                <state_interface name="effort"/> <!-- current -->
             </joint>
-            <joint name="finger_c">
-                <command_interface name="position"/>
+            <joint name="finger_1_joint_3">
                 <state_interface name="position"/>
-                <state_interface name="velocity"/>
-                <state_interface name="effort"/> <!-- current -->
             </joint>
+            <joint name="finger_2_joint_1">
+                <state_interface name="position"/>
+            </joint>
+            <joint name="finger_2_joint_2">
+                <state_interface name="position"/>
+            </joint>
+            <joint name="finger_2_joint_3">
+                <state_interface name="position"/>
+            </joint>
+            <joint name="finger_3_joint_1">
+                <state_interface name="position"/>
+            </joint>
+            <joint name="finger_3_joint_2">
+                <state_interface name="position"/>
+            </joint>
+            <joint name="finger_3_joint_3">
+                <state_interface name="position"/>
+            </joint>
+            <joint name="palm_finger_1_joint">
+                <state_interface name="position"/>
+            </joint>
+            <joint name="palm_finger_2_joint">
+                <state_interface name="position"/>
+            </joint>
+            <!-- since the robotiq 3f is underactuated, we use transmissions to defined how the motors
+                    are connected to the joints. -->
+            <transmission name="individual_control_transmission">
+                <!-- TODO which package should this live in? -->
+                <plugin>robotiq_3f_driver/IndividualControlTransmission</plugin>
+                <!-- TODO I wish I didn't have to list these here, it's duplicated in the plugin -->
+                <actuator name="finger_a_actuator" role="finger_a_actuator"/>
+                <actuator name="finger_b_actuator" role="finger_b_actuator"/>
+                <actuator name="finger_c_actuator" role="finger_c_actuator"/>
+                <actuator name="scissor_actuator" role="scissor_actuator"/>
+                <joint name="finger_1_joint_1" role="finger_1_joint_1"/>
+                <joint name="finger_1_joint_2" role="finger_1_joint_2"/>
+                <joint name="finger_1_joint_3" role="finger_1_joint_3"/>
+                <joint name="finger_2_joint_1" role="finger_2_joint_1"/>
+                <joint name="finger_2_joint_2" role="finger_2_joint_2"/>
+                <joint name="finger_2_joint_3" role="finger_2_joint_3"/>
+                <joint name="finger_3_joint_1" role="finger_3_joint_1"/>
+                <joint name="finger_3_joint_2" role="finger_3_joint_2"/>
+                <joint name="finger_3_joint_3" role="finger_3_joint_3"/>
+                <joint name="palm_finger_1_joint" role="palm_finger_1_joint"/>
+                <joint name="palm_finger_2_joint" role="palm_finger_2_joint"/>
+            </transmission>
         </ros2_control>
     </xacro:macro>

File: robotiq_3f_description/urdf/robotiq_3f_gripper.xacro (robot description, xacro)
@@ -1,5 +1,6 @@
 <?xml version="1.0"?>
 <robot name="example_robot" xmlns:xacro="http://www.ros.org/wiki/xacro">
+  <xacro:arg name="usb_port" default="/dev/ttyUSB1"/>
   <xacro:include filename="$(find robotiq_3f_description)/urdf/robotiq_3f_gripper_macro.xacro"/>
-  <xacro:robotiq_3f_gripper use_fake_hardware="false"/>
+  <xacro:robotiq_3f_gripper use_fake_hardware="false" usb_port="$(arg usb_port)"/>
 </robot>

File: robotiq_3f_description/urdf/robotiq_3f_gripper_macro.xacro (robot description, xacro)
@@ -13,5 +13,5 @@
         <xacro:robotiq_3f_gripper_finger_articulated prefix="${prefix}finger_1_"/>
         <xacro:robotiq_3f_gripper_finger_articulated prefix="${prefix}finger_2_"/>
-        <xacro:robotiq_3f_gripper_finger_articulated prefix="${prefix}finger_middle_"/>
+        <xacro:robotiq_3f_gripper_finger_articulated prefix="${prefix}finger_3_"/>
         <!-- link list -->
         <link name="${prefix}palm">
@@ -55,7 +55,7 @@
             <limit lower="-0.192" upper="0.1784" effort="100" velocity="100"/>
         </joint>
-        <joint name="${prefix}palm_finger_middle_joint" type="fixed">
+        <joint name="${prefix}palm_finger_3_joint" type="fixed">
             <parent link="${prefix}palm"/>
-            <child link="${prefix}finger_middle_link_0"/>
+            <child link="${prefix}finger_3_link_0"/>
             <axis xyz="0 0 1"/>
             <origin xyz="0.0455 0.0214 0" rpy="0 0 1.57"/>

Commit message: rename finger_1/2/3 to match finger_a/b/c
looks good in rviz.
removed a bunch of uncesseary info from the ros2_control.xacro

File: robotiq_3f_description/urdf/robotiq_3f_driver_ros2_control.xacro (robot description, xacro)
@@ -20,59 +20,12 @@
                 <param name="slave_address">${slave_address}</param>
             </hardware>
-            <!-- NOTE should we also have position and velocity interfaces? -->
-            <joint name="finger_1_joint_1">
-                <state_interface name="position"/>
-            </joint>
-            <joint name="finger_1_joint_2">
-                <state_interface name="position"/>
-            </joint>
-            <joint name="finger_1_joint_3">
-                <state_interface name="position"/>
-            </joint>
-            <joint name="finger_2_joint_1">
-                <state_interface name="position"/>
-            </joint>
-            <joint name="finger_2_joint_2">
-                <state_interface name="position"/>
-            </joint>
-            <joint name="finger_2_joint_3">
-                <state_interface name="position"/>
-            </joint>
-            <joint name="finger_3_joint_1">
-                <state_interface name="position"/>
-            </joint>
-            <joint name="finger_3_joint_2">
-                <state_interface name="position"/>
-            </joint>
-            <joint name="finger_3_joint_3">
-                <state_interface name="position"/>
-            </joint>
-            <joint name="palm_finger_1_joint">
-                <state_interface name="position"/>
-            </joint>
-            <joint name="palm_finger_2_joint">
-                <state_interface name="position"/>
-            </joint>
-            <!-- since the robotiq 3f is underactuated, we use transmissions to defined how the motors
-                    are connected to the joints. -->
+            <!--
+                since the robotiq 3f is underactuated, we use transmissions to defined how the motors
+                are connected to the joints.
+                We therefore also do not list the joints and their state/command interfaces here,
+                because all that information is contained in the hardware interface.
+            -->
             <transmission name="individual_control_transmission">
-                <!-- TODO which package should this live in? -->
-                <plugin>robotiq_3f_driver/IndividualControlTransmission</plugin>
-                <!-- TODO I wish I didn't have to list these here, it's duplicated in the plugin -->
-                <actuator name="finger_a_actuator" role="finger_a_actuator"/>
-                <actuator name="finger_b_actuator" role="finger_b_actuator"/>
-                <actuator name="finger_c_actuator" role="finger_c_actuator"/>
-                <actuator name="scissor_actuator" role="scissor_actuator"/>
-                <joint name="finger_1_joint_1" role="finger_1_joint_1"/>
-                <joint name="finger_1_joint_2" role="finger_1_joint_2"/>
-                <joint name="finger_1_joint_3" role="finger_1_joint_3"/>
-                <joint name="finger_2_joint_1" role="finger_2_joint_1"/>
-                <joint name="finger_2_joint_2" role="finger_2_joint_2"/>
-                <joint name="finger_2_joint_3" role="finger_2_joint_3"/>
-                <joint name="finger_3_joint_1" role="finger_3_joint_1"/>
-                <joint name="finger_3_joint_2" role="finger_3_joint_2"/>
-                <joint name="finger_3_joint_3" role="finger_3_joint_3"/>
-                <joint name="palm_finger_1_joint" role="palm_finger_1_joint"/>
-                <joint name="palm_finger_2_joint" role="palm_finger_2_joint"/>
+                <plugin>robotiq_3f_transmission_plugins/IndividualControlTransmission</plugin>
             </transmission>
         </ros2_control>

File: robotiq_3f_description/urdf/robotiq_3f_gripper_finger_macro.xacro (robot description, xacro)
@@ -2,6 +2,5 @@
 robotiq_3f_gripper_finder_articulated_macro(prefix)
 Creates an articulated robotiq_3f_gripper finder with the passed in prefix.  The
-prefix typcially includes the hand prefix and an identifier for the
-finger(i.e. finger_1, etc...).
+prefix typcially includes the hand prefix and an identifier for the finger
 -->
 <robot xmlns:xacro="http://ros.org/wiki/xacro">

File: robotiq_3f_description/urdf/robotiq_3f_gripper_macro.xacro (robot description, xacro)
@@ -11,7 +11,7 @@
                 use_fake_hardware="${use_fake_hardware}"
                 usb_port="${usb_port}"/>
-        <xacro:robotiq_3f_gripper_finger_articulated prefix="${prefix}finger_1_"/>
-        <xacro:robotiq_3f_gripper_finger_articulated prefix="${prefix}finger_2_"/>
-        <xacro:robotiq_3f_gripper_finger_articulated prefix="${prefix}finger_3_"/>
+        <xacro:robotiq_3f_gripper_finger_articulated prefix="${prefix}finger_b_"/>
+        <xacro:robotiq_3f_gripper_finger_articulated prefix="${prefix}finger_a_"/>
+        <xacro:robotiq_3f_gripper_finger_articulated prefix="${prefix}finger_c_"/>
         <!-- link list -->
         <link name="${prefix}palm">
@@ -41,21 +41,21 @@
         <!-- end of link list -->
         <!-- joint list -->
-        <joint name="${prefix}palm_finger_1_joint" type="revolute">
+        <joint name="${prefix}palm_finger_c_joint" type="revolute">
             <parent link="${prefix}palm"/>
-            <child link="${prefix}finger_1_link_0"/>
+            <child link="${prefix}finger_c_link_0"/>
             <axis xyz="0 1 0"/>
             <origin xyz="-0.0455 0.0214 0.036" rpy="0 3.1416 -1.57"/>
             <limit lower="-0.1784" upper="0.192" effort="100" velocity="100"/>
         </joint>
-        <joint name="${prefix}palm_finger_2_joint" type="revolute">
+        <joint name="${prefix}palm_finger_b_joint" type="revolute">
             <parent link="${prefix}palm"/>
-            <child link="${prefix}finger_2_link_0"/>
+            <child link="${prefix}finger_b_link_0"/>
             <axis xyz="0 1 0"/>
             <origin xyz="-0.0455 0.0214 -0.036" rpy="0 3.1416 -1.57"/>
             <limit lower="-0.192" upper="0.1784" effort="100" velocity="100"/>
         </joint>
-        <joint name="${prefix}palm_finger_3_joint" type="fixed">
+        <joint name="${prefix}palm_finger_a_joint" type="fixed">
             <parent link="${prefix}palm"/>
-            <child link="${prefix}finger_3_link_0"/>
+            <child link="${prefix}finger_a_link_0"/>
             <axis xyz="0 0 1"/>
             <origin xyz="0.0455 0.0214 0" rpy="0 0 1.57"/>
